File: KiCad/V0-PT100.sch (KiCad schematic (older format))
At the start: 0 parts

Commit message: Inital PT100 Adapter schematic
Parts:
- added C? (x2): 10uF, symbol Device:C
- added C? (x2): 10uF, symbol Device:C_Small
- added D? (x3): 1N4148, Diode_THT:D_DO-35_SOD27_P7.62mm_Horizontal, symbol Diode:1N4148
- added FB?: Ferrite_Bead_Small, symbol Device:Ferrite_Bead_Small
- added J?: SPI1, symbol Connector_Generic:Conn_02x03_Odd_Even
- added J?: E0-Stop, symbol Connector_Generic:Conn_02x01
- added J?: T1, symbol Connector:Screw_Terminal_01x02
- added J?: T2, symbol Connector:Screw_Terminal_01x02
- added JP?: SolderJumper_3_Bridged12, symbol Jumper:SolderJumper_3_Bridged12
- added JP? (x2): SolderJumper_2_Bridged, symbol Jumper:SolderJumper_2_Bridged
- added R?: 430, symbol Device:R_Small_US
- added R? (x3): 10K, symbol Device:R_Small_US
- added U?: MAX31865ATP_, digikey-footprints:TQFN-20-1EP_5x5mm, symbol V0PT100:MAX31865ATP_
- added U?: MIC5225-3.3YM5-TR, SOT-23-5_M5_MCH, symbol V0PT100:MIC5225-3.3YM5-TR
Connections:
- net labels added: +3.3V, +5V, BIAS, CS, FORCE+, FORCE-, GND, M-FORCE+, M-FORCE-, M-FORCE2, M-RTDIN+, M-RTDIN-, MISO, MOSI, RST, RTDIN-, SCK
- wire segments 0 -> 105
- no-connect marks 0 -> 1

Commit message: Schematic Updates. Next Up PCB layout
Parts:
- removed U?: MAX31865ATP_, digikey-footprints:TQFN-20-1EP_5x5mm, symbol V0PT100:MAX31865ATP_
- added U1: MAX31865ATP+, V0PT100:MAX31865ATP&plus_, symbol V0PT100:MAX31865ATP+
- C1, C2, C3, C4: renamed from C?; footprint (none) -> V0PT100:C_0603_1608Metric_Pad1.05x0.95mm_HandSolder
- D1, D2, D3: renamed from D?; footprint Diode_THT:D_DO-35_SOD27_P7.62mm_Horizontal -> Diode_SMD:D_SOD-323
- FB1: renamed from FB?; footprint (none) -> V0PT100:L_0603_1608Metric_Pad1.05x0.95mm_HandSolder
- J1, J2, J4: renamed from J?; footprint (none) -> Connector_PinHeader_2.54mm:PinHeader_1x02_P2.54mm_Horizontal
- J3: renamed from J?; footprint (none) -> Connector_PinHeader_2.54mm:PinHeader_2x03_P2.54mm_Horizontal
- JP1: renamed from JP?; footprint (none) -> V0PT100:SolderJumper-3_P1.3mm_Bridged12_RoundedPad1.0x1.5mm
- JP2, JP3: renamed from JP?; footprint (none) -> V0PT100:SolderJumper-2_P1.3mm_Bridged_RoundedPad1.0x1.5mm
- R1, R2, R3, R4: renamed from R?; footprint (none) -> V0PT100:R_0603_1608Metric_Pad1.05x0.95mm_HandSolder
- U2: renamed from U?; footprint SOT-23-5_M5_MCH -> V0PT100:MIC5225-3.3YM5-TR
Connections:
- net labels added: M-CS, M-SCK, M-SDI, SDI, SDO
- net labels removed: BIAS, MISO, MOSI
- wire segments 105 -> 109
Other:
- moved on the sheet: C1, C2, C3, C4, D1, D2, D3, FB1, J3, JP1, JP2, JP3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

Commit message: Swap out some component
Parts:
- removed J1: T1, Connector_PinHeader_2.54mm:PinHeader_1x02_P2.54mm_Horizontal, symbol Connector:Screw_Terminal_01x02
- removed J2: T2, Connector_PinHeader_2.54mm:PinHeader_1x02_P2.54mm_Horizontal, symbol Connector:Screw_Terminal_01x02
- removed J4: E0-Stop, Connector_PinHeader_2.54mm:PinHeader_1x02_P2.54mm_Horizontal, symbol Connector_Generic:Conn_02x01
- added J1: T1, V0PT100:1984617, symbol V0PT100:1984617
- added J2: T2, V0PT100:1984617, symbol V0PT100:1984617
- added J4: Servos, Connector_PinSocket_2.54mm:PinSocket_1x03_P2.54mm_Vertical, symbol Connector_Generic:Conn_01x03
- J3: footprint Connector_PinHeader_2.54mm:PinHeader_2x03_P2.54mm_Horizontal -> Connector_PinSocket_2.54mm:PinSocket_2x03_P2.54mm_Vertical
Connections:
- no-connect marks 1 -> 2
Changed lines of the file:
@@
 F 0 "J3" H 7100 1917 50  0000 C CNN
 F 1 "SPI1" H 7100 1826 50  0000 C CNN
-F 2 "Connector_PinHeader_2.54mm:PinHeader_2x03_P2.54mm_Horizontal" H 7050 1600 50  0001 C CNN
+F 2 "Connector_PinSocket_2.54mm:PinSocket_2x03_P2.54mm_Vertical" H 7050 1600 50  0001 C CNN
 F 3 "~" H 7050 1600 50  0001 C CNN
 	1    7050 1600
-	1    0    0    -1
-$EndComp
-$Comp
-L Connector_Generic:Conn_02x01 J4
-U 1 1 5F13421A
-P 7050 2100
-F 0 "J4" H 7100 2317 50  0000 C CNN
-F 1 "E0-Stop" H 7100 2226 50  0000 C CNN
-F 2 "Connector_PinHeader_2.54mm:PinHeader_1x02_P2.54mm_Horizontal" H 7050 2100 50  0001 C CNN
-F 3 "~" H 7050 2100 50  0001 C CNN
-	1    7050 2100
 	1    0    0    -1
 $EndComp
@@
 	0    -1   -1   0
 $EndComp
-Wire Wire Line
-	6850 2100 6500 2100
 $Comp
 L power:GND #PWR0104
 U 1 1 5F13BFF4
-P 6500 2100
-F 0 "#PWR0104" H 6500 1850 50  0001 C CNN
-F 1 "GND" V 6505 1972 50  0000 R CNN
-F 2 "" H 6500 2100 50  0001 C CNN
-F 3 "" H 6500 2100 50  0001 C CNN
-	1    6500 2100
-	0    1    1    0
-$EndComp
-Wire Wire Line
-	7350 2100 7700 2100
-Text Label 7550 2100 0    50   ~ 0
-CS
+P 6500 2050
+F 0 "#PWR0104" H 6500 1800 50  0001 C CNN
+F 1 "GND" V 6505 1922 50  0000 R CNN
+F 2 "" H 6500 2050 50  0001 C CNN
+F 3 "" H 6500 2050 50  0001 C CNN
+	1    6500 2050
+	0    1    1    0
+$EndComp
 $Comp
 L V0PT100:MIC5225-3.3YM5-TR U2
@@
 	7250 3450 7250 3650
 Connection ~ 7300 2850
-$Comp
-L Connector:Screw_Terminal_01x02 J1
-U 1 1 5F1B5E11
-P 5250 4900
-F 0 "J1" H 5168 4575 50  0000 C CNN
-F 1 "T1" H 5168 4666 50  0000 C CNN
-F 2 "Connector_PinHeader_2.54mm:PinHeader_1x02_P2.54mm_Horizontal" H 5250 4900 50  0001 C CNN
-F 3 "~" H 5250 4900 50  0001 C CNN
-	1    5250 4900
-	1    0    0    1
-$EndComp
-$Comp
-L Connector:Screw_Terminal_01x02 J2
-U 1 1 5F1B8A31
-P 5250 5350
-F 0 "J2" H 5168 5025 50  0000 C CNN
-F 1 "T2" H 5168 5116 50  0000 C CNN
-F 2 "Connector_PinHeader_2.54mm:PinHeader_1x02_P2.54mm_Horizontal" H 5250 5350 50  0001 C CNN
-F 3 "~" H 5250 5350 50  0001 C CNN
-	1    5250 5350
-	1    0    0    1
-$EndComp
 Text Label 4600 4800 0    50   ~ 0
 FORCE+
@@
 Wire Wire Line
 	4500 3450 4650 3450
+$Comp
+L Connector_Generic:Conn_01x03 J4
+U 1 1 5F4C2A3A
+P 7050 2150
+F 0 "J4" H 7130 2192 50  0000 L CNN
+F 1 "Servos" H 7130 2101 50  0000 L CNN
+F 2 "Connector_PinSocket_2.54mm:PinSocket_1x03_P2.54mm_Vertical" H 7050 2150 50  0001 C CNN
+F 3 "~" H 7050 2150 50  0001 C CNN
+	1    7050 2150
+	1    0    0    -1
+$EndComp
+Wire Wire Line
+	6850 2050 6500 2050
+Wire Wire Line
+	6850 2250 6500 2250
+NoConn ~ 6850 2150
+Text Label 6550 2250 0    50   ~ 0
+CS
+$Comp
+L V0PT100:1984617 J1
+U 1 1 5F4F4DC1
+P 5050 4900
+F 0 "J1" H 5292 4619 60  0000 C CNN
+F 1 "T1" H 5292 4619 60  0001 C CNN
+F 2 "V0PT100:1984617" H 5450 4840 60  0001 C CNN
+F 3 "" H 5050 4900 60  0000 C CNN
+	1    5050 4900
+	1    0    0    1
+$EndComp
+$Comp
+L V0PT100:1984617 J2
+U 1 1 5F4F5EA2
+P 5050 5350
+F 0 "J2" H 5292 5069 60  0000 C CNN
+F 1 "T2" H 5292 5069 60  0001 C CNN
+F 2 "V0PT100:1984617" H 5450 5290 60  0001 C CNN
+F 3 "" H 5050 5350 60  0000 C CNN
+	1    5050 5350
+	1    0    0    1
+$EndComp
 $EndSCHEMATC

Commit message: Inital PCB layout complete
Parts:
- removed J4: Servos, Connector_PinSocket_2.54mm:PinSocket_1x03_P2.54mm_Vertical, symbol Connector_Generic:Conn_01x03
- added J4: Output, Connector_PinHeader_2.54mm:PinHeader_1x01_P2.54mm_Horizontal, symbol Connector:Conn_01x01_Male
Connections:
- net labels added: BIAS, DVDD, ISENSOR, REFIN+, REFIN-, VDD
- wire segments 109 -> 107
- no-connect marks 2 -> 1
Changed lines of the file:
@@
-$EndComp
-$Comp
-L power:GND #PWR0104
-U 1 1 5F13BFF4
-P 6500 2050
-F 0 "#PWR0104" H 6500 1800 50  0001 C CNN
-F 1 "GND" V 6505 1922 50  0000 R CNN
-F 2 "" H 6500 2050 50  0001 C CNN
-F 3 "" H 6500 2050 50  0001 C CNN
-	1    6500 2050
-	0    1    1    0
 $EndComp
 $Comp
@@
 $EndComp
 Wire Wire Line
-	2100 2200 2350 2200
-Wire Wire Line
-	2350 2200 2350 2250
-Wire Wire Line
-	2350 2250 2500 2250
-Wire Wire Line
-	2100 2000 2400 2000
-Wire Wire Line
-	2400 2000 2400 1950
-Wire Wire Line
-	2400 1950 2500 1950
-Wire Wire Line
 	2500 2150 2400 2150
 Wire Wire Line
-	2400 2150 2400 2000
-Connection ~ 2400 2000
-Wire Wire Line
 	2500 1850 1850 1850
 Wire Wire Line
 	1850 1850 1850 2250
-Wire Wire Line
-	1850 2250 2350 2250
-Connection ~ 2350 2250
 Wire Wire Line
 	7050 3250 7850 3250
@@
 Wire Wire Line
 	4500 3450 4650 3450
-$Comp
-L Connector_Generic:Conn_01x03 J4
-U 1 1 5F4C2A3A
-P 7050 2150
-F 0 "J4" H 7130 2192 50  0000 L CNN
-F 1 "Servos" H 7130 2101 50  0000 L CNN
-F 2 "Connector_PinSocket_2.54mm:PinSocket_1x03_P2.54mm_Vertical" H 7050 2150 50  0001 C CNN
-F 3 "~" H 7050 2150 50  0001 C CNN
-	1    7050 2150
-	1    0    0    -1
-$EndComp
-Wire Wire Line
-	6850 2050 6500 2050
-Wire Wire Line
-	6850 2250 6500 2250
-NoConn ~ 6850 2150
-Text Label 6550 2250 0    50   ~ 0
+Wire Wire Line
+	7250 2200 6900 2200
+Text Label 6950 2200 0    50   ~ 0
 CS
 $Comp
 L V0PT100:1984617 J1
 U 1 1 5F4F4DC1
-P 5050 4900
-F 0 "J1" H 5292 4619 60  0000 C CNN
-F 1 "T1" H 5292 4619 60  0001 C CNN
-F 2 "V0PT100:1984617" H 5450 4840 60  0001 C CNN
-F 3 "" H 5050 4900 60  0000 C CNN
-	1    5050 4900
-	1    0    0    1
+P 5050 4800
+F 0 "J1" H 5292 4519 60  0000 C CNN
+F 1 "T1" H 5292 4519 60  0001 C CNN
+F 2 "V0PT100:1984617" H 5450 4740 60  0001 C CNN
+F 3 "" H 5050 4800 60  0000 C CNN
+	1    5050 4800
+	1    0    0    -1
 $EndComp
 $Comp
 L V0PT100:1984617 J2
 U 1 1 5F4F5EA2
-P 5050 5350
-F 0 "J2" H 5292 5069 60  0000 C CNN
-F 1 "T2" H 5292 5069 60  0001 C CNN
-F 2 "V0PT100:1984617" H 5450 5290 60  0001 C CNN
-F 3 "" H 5050 5350 60  0000 C CNN
-	1    5050 5350
-	1    0    0    1
-$EndComp
+P 5050 5250
+F 0 "J2" H 5292 4969 60  0000 C CNN
+F 1 "T2" H 5292 4969 60  0001 C CNN
+F 2 "V0PT100:1984617" H 5450 5190 60  0001 C CNN
+F 3 "" H 5050 5250 60  0000 C CNN
+	1    5050 5250
+	1    0    0    -1
+$EndComp
+$Comp
+L Connector:Conn_01x01_Male J4
+U 1 1 5F138E11
+P 6700 2200
+F 0 "J4" H 6808 2381 50  0000 C CNN
+F 1 "Output" H 6800 2300 50  0000 C CNN
+F 2 "Connector_PinHeader_2.54mm:PinHeader_1x01_P2.54mm_Horizontal" H 6700 2200 50  0001 C CNN
+F 3 "~" H 6700 2200 50  0001 C CNN
+	1    6700 2200
+	1    0    0    -1
+$EndComp
+Text Label 2200 1850 0    50   ~ 0
+BIAS
+Wire Wire Line
+	2500 2250 2100 2250
+Wire Wire Line
+	2100 2250 2100 2200
+Wire Wire Line
+	1850 2250 2100 2250
+Connection ~ 2100 2250
+Text Label 2200 2250 0    50   ~ 0
+REFIN+
+Wire Wire Line
+	2500 1950 2100 1950
+Wire Wire Line
+	2100 1950 2100 2000
+Wire Wire Line
+	2400 2150 2400 2000
+Wire Wire Line
+	2400 2000 2100 2000
+Connection ~ 2100 2000
+Text Label 2200 1950 0    50   ~ 0
+ISENSOR
+Text Label 2400 2150 0    50   ~ 0
+REFIN-
+Text Label 2200 1750 0    50   ~ 0
+GND
+Text Label 2350 3550 0    50   ~ 0
+VDD
+Text Label 2350 3450 0    50   ~ 0
+DVDD
 $EndSCHEMATC

Commit message: Add files via upload
Parts:
- C1, C2: symbol Device:C_Small -> V0-PT100-rescue:C_Small-Device
- C3, C4: symbol Device:C -> V0-PT100-rescue:C-Device
- D1, D2, D3: symbol Diode:1N4148 -> V0-PT100-rescue:1N4148-Diode
- FB1: symbol Device:Ferrite_Bead_Small -> V0-PT100-rescue:Ferrite_Bead_Small-Device
- J3: symbol Connector_Generic:Conn_02x03_Odd_Even -> V0-PT100-rescue:Conn_02x03_Odd_Even-Connector_Generic
- J4: symbol Connector:Conn_01x01_Male -> V0-PT100-rescue:Conn_01x01_Male-Connector
- JP1: symbol Jumper:SolderJumper_3_Bridged12 -> V0-PT100-rescue:SolderJumper_3_Bridged12-Jumper
- JP2, JP3: symbol Jumper:SolderJumper_2_Bridged -> V0-PT100-rescue:SolderJumper_2_Bridged-Jumper
- R1, R2, R3, R4: symbol Device:R_Small_US -> V0-PT100-rescue:R_Small_US-Device
Changed lines of the file:
@@
 $EndDescr
 $Comp
-L Device:R_Small_US R3
+L V0-PT100-rescue:R_Small_US-Device R3
 U 1 1 5F129B4A
 P 2100 2100
@@
 $EndComp
 $Comp
-L Connector_Generic:Conn_02x03_Odd_Even J3
+L V0-PT100-rescue:Conn_02x03_Odd_Even-Connector_Generic J3
 U 1 1 5F132E40
 P 7050 1600
@@
 	7350 1500 7700 1500
 $Comp
-L power:+5V #PWR0102
+L V0-PT100-rescue:+5V-power #PWR0102
 U 1 1 5F138591
 P 7700 1500
@@
 	7350 1700 7700 1700
 $Comp
-L power:GND #PWR0103
+L V0-PT100-rescue:GND-power #PWR0103
 U 1 1 5F13AEF8
 P 7700 1700
@@
 $EndComp
 $Comp
-L power:+5V #PWR0105
+L V0-PT100-rescue:+5V-power #PWR0105
 U 1 1 5F14C31B
 P 6150 4700
@@
 $EndComp
 $Comp
-L power:GND #PWR0106
+L V0-PT100-rescue:GND-power #PWR0106
 U 1 1 5F14CC74
 P 6150 5250
@@
 	6150 5150 6150 5250
 $Comp
-L Device:C C3
+L V0-PT100-rescue:C-Device C3
 U 1 1 5F14D857
 P 6150 5000
@@
 NoConn ~ 8600 5150
 $Comp
-L Device:C C4
+L V0-PT100-rescue:C-Device C4
 U 1 1 5F1563E9
 P 8800 5300
@@
 $EndComp
 $Comp
-L power:GND #PWR0108
+L V0-PT100-rescue:GND-power #PWR0108
 U 1 1 5F15678F
 P 8800 5650
@@
 Connection ~ 8800 5050
 $Comp
-L Device:Ferrite_Bead_Small FB1
+L V0-PT100-rescue:Ferrite_Bead_Small-Device FB1
 U 1 1 5F16051D
 P 1950 3550
@@
 $EndComp
 $Comp
-L Device:C_Small C2
+L V0-PT100-rescue:C_Small-Device C2
 U 1 1 5F164BA8
 P 2150 3700
@@
 $EndComp
 $Comp
-L Device:C_Small C1
+L V0-PT100-rescue:C_Small-Device C1
 U 1 1 5F1656B5
 P 2150 3200
@@
 $EndComp
 $Comp
-L Diode:1N4148 D1
+L V0-PT100-rescue:1N4148-Diode D1
 U 1 1 5F1898C2
 P 6900 2650
@@
 $EndComp
 $Comp
-L Diode:1N4148 D2
+L V0-PT100-rescue:1N4148-Diode D2
 U 1 1 5F18BFA0
 P 6900 2950
@@
 $EndComp
 $Comp
-L Diode:1N4148 D3
+L V0-PT100-rescue:1N4148-Diode D3
 U 1 1 5F18DB50
 P 6900 3250
@@
 $EndComp
 $Comp
-L Device:R_Small_US R1
+L V0-PT100-rescue:R_Small_US-Device R1
 U 1 1 5F19BEFC
 P 7250 3750
@@
 $EndComp
 $Comp
-L Device:R_Small_US R2
+L V0-PT100-rescue:R_Small_US-Device R2
 U 1 1 5F19D211
 P 7550 3750
@@
 $EndComp
 $Comp
-L Device:R_Small_US R4
+L V0-PT100-rescue:R_Small_US-Device R4
 U 1 1 5F19DE82
 P 7850 3750
@@
 M-FORCE-
 $Comp
-L Jumper:SolderJumper_3_Bridged12 JP1
+L V0-PT100-rescue:SolderJumper_3_Bridged12-Jumper JP1
 U 1 1 5F2A911F
 P 2550 4750
@@
 	2950 4550 2950 4700
 $Comp
-L power:GND #PWR0114
+L V0-PT100-rescue:GND-power #PWR0114
 U 1 1 5F2B1C1D
 P 2550 5050
@@
 	3050 5100 3850 5100
 $Comp
-L Jumper:SolderJumper_2_Bridged JP2
+L V0-PT100-rescue:SolderJumper_2_Bridged-Jumper JP2
 U 1 1 5F2D5027
 P 3850 4900
@@
 $EndComp
 $Comp
-L Jumper:SolderJumper_2_Bridged JP3
+L V0-PT100-rescue:SolderJumper_2_Bridged-Jumper JP3
 U 1 1 5F2D59C1
 P 3950 5400
@@
 $EndComp
 $Comp
-L power:GND #PWR0109
+L V0-PT100-rescue:GND-power #PWR0109
 U 1 1 5F3FBEBB
 P 1900 3700
@@
 $EndComp
 $Comp
-L power:GND #PWR0110
+L V0-PT100-rescue:GND-power #PWR0110
 U 1 1 5F3FD6B1
 P 1900 3200
@@
 Connection ~ 4500 3450
 $Comp
-L power:GND #PWR0111
+L V0-PT100-rescue:GND-power #PWR0111
 U 1 1 5F43200D
 P 2150 1750
@@
 	2500 1750 2150 1750
 $Comp
-L power:GND #PWR0112
+L V0-PT100-rescue:GND-power #PWR0112
 U 1 1 5F43897B
 P 4650 3450
@@
 $EndComp
 $Comp
-L Connector:Conn_01x01_Male J4
+L V0-PT100-rescue:Conn_01x01_Male-Connector J4
 U 1 1 5F138E11
 P 6700 2200
